File: sks.kicad_pcb (KiCad board)
At the start: 2 copper layers, 34 x 28 mm, 18 parts, among them J1 Conn_01x03, Q1 BC847, U1 Opto_Interrupter, U2 NE555

Commit message: 2019.05.12
Parts:
- added C4: 0.1, Capacitor_SMD:C_0805_2012Metric_Pad1.15x1.40mm_HandSolder, F.Cu at (111.0, 52.2)
- added R7: 10k, Resistor_SMD:R_0805_2012Metric_Pad1.15x1.40mm_HandSolder, F.Cu at (114.2, 51.1)
- C1, C2, C3: value C -> 0.1
- D1: value D -> BAS32
- J1: footprint Connector_Molex:Molex_Micro-Latch_53253-0370_1x03_P2.00mm_Vertical -> Connector_Molex:Molex_KK-254_AE-6410-03A_1x03_P2.54mm_Vertical
- R2: value 10k -> 100k
- R4: value R -> 10k*
- R5: value R -> 100k
- R6: value R -> 100
- moved J1 3.92 mm to (126.2, 46.8), turned to 90 degrees
- moved D1 0.76 mm to (122.0, 44.9)
- moved R3 0.46 mm to (108.0, 51.1)
Connections:
- Q1 pad 3: Net-(Q1-Pad3) -> Net-(C4-Pad2)
- R3 pad 2: Net-(Q1-Pad3) -> Net-(C4-Pad2)
- U2 pad 2: Net-(Q1-Pad3) -> Net-(C4-Pad1)
Routing:
- net Net-(Q1-Pad3): track 13.9 -> 0.00 mm
- net /OUT: track 8.86 -> 18.4 mm
- net Net-(C4-Pad1): track 0.00 -> 6.79 mm
- net Net-(C4-Pad2): track 0.00 -> 5.11 mm
- net Net-(D1-Pad2): track 3.36 -> 7.88 mm
